File: electrobadge/airbox.kicad_pcb (KiCad board)
At the start: 2 copper layers, 79 x 36.8 mm, 49 parts, among them J1 SEN66, J10 MEZ_SIGNALS, J2 MCU-CONN-1, J3 SOLAR, J4 BATTERY, J5 SCD30, J6 MCU-CONN-2, J7 Conn_01x03, J9 MEZ_SIGNALS, Q1 AO3401A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

Commit message: Badge finish
Other:
- outline, holes or cut-outs redrawn
- board text added: "Alacrity Airbox Bootcamp"
- board text removed: "Alacrity AirBox V2-rc1"
- board text removed: "CHARGER BYPASS"
