File: electronics/DAUGHTERBOARD_DIGITS.kicad_sch (KiCad schematic)
At the start: 19 parts, among them J11 MEZ_SIGNALS, J12 MEZ_SIGNALS, Q2 AO3400A, Q3 AO3400A, U4 GS2022CW-G, U5 74HC157, U6 HEF4543B, U7 74LVC1GU04DRL, U8 74HC595, U9 74LVC1GU04DRL

Commit message: Route PCB for demo powerstage
Parts:
- C1: LCSC (none) -> C57112
- C11, C12, C2: LCSC (none) -> C14663
- R1, R2: LCSC (none) -> C22787
- R3: LCSC (none) -> C22807
Changed lines of the file:
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@@
+			)
+		)
+		(property "LCSC" "C14663"
+			(at 81.28 41.91 90)
+			(hide yes)
+			(show_name no)
+			(do_not_autoplace no)
+			(effects
+				(font
+					(size 1.27 1.27)
+				)
 			)
 		)
@@
 			)
 		)
+		(property "LCSC" "C14663"
+			(at 139.7 46.99 90)
+			(hide yes)
+			(show_name no)
+			(do_not_autoplace no)
+			(effects
+				(font
+					(size 1.27 1.27)
+				)
+			)
+		)
 		(pin "1"
 		)
@@
 			)
 		)
+		(property "LCSC" "C57112"
+			(at 38.1 120.65 90)
+			(hide yes)
+			(show_name no)
+			(do_not_autoplace no)
+			(effects
+				(font
+					(size 1.27 1.27)
+				)
+			)
+		)
 		(pin "1"
 		)
@@
 			)
 		)
+		(property "LCSC" "C22807"
+			(at 67.31 108.712 90)
+			(hide yes)
+			(show_name no)
+			(do_not_autoplace no)
+			(effects
+				(font
+					(size 1.27 1.27)
+				)
+			)
+		)
 		(pin "2"
 		)
@@
 		(property "Description" "Unpolarized capacitor"
 			(at 111.76 48.26 0)
+			(hide yes)
+			(show_name no)
+			(do_not_autoplace no)
+			(effects
+				(font
+					(size 1.27 1.27)
+				)
+			)
+		)
+		(property "LCSC" "C14663"
+			(at 111.76 43.18 90)
 			(hide yes)
 			(show_name no)
@@
 			)
 		)
+		(property "LCSC" "C22787"
+			(at 228.6 100.33 90)
+			(hide yes)
+			(show_name no)
+			(do_not_autoplace no)
+			(effects
+				(font
+					(size 1.27 1.27)
+				)
+			)
+		)
 		(pin "2"
 		)
@@
 			(hide yes)
 			(show_name no)
+			(do_not_autoplace no)
+			(effects
+				(font
+					(size 1.27 1.27)
+				)
+			)
+		)
+		(property "LCSC" "C22787"
+			(at 199.39 100.33 90)
+			(hide yes)
+			(show_name no)
